File: power_splitter/resistive-power-splitter.sch (KiCad schematic (older format))
At the start: 36 parts, among them J1 Conn_01x02, J10 Conn_01x02, J11 Conn_01x02, J12 Conn_01x02, J2 Conn_01x02, J3 Conn_01x02, J4 Conn_01x02, J5 Conn_01x02, J6 Conn_01x02, J7 Conn_01x02, J8 Conn_01x02, J9 Conn_01x02

Commit message: power splitter: footprint assignment & parts placement
Parts:
- J1, J10, J11, J12, J2, J3, J4, J5, J6, J7, J8, J9: footprint (none) -> Connector_Coaxial:SMA_Amphenol_132203-12_Horizontal
Changed lines of the file:
@@
 F 0 "J1" H 1568 1125 50  0000 C CNN
 F 1 "Conn_01x02" H 1568 1216 50  0000 C CNN
-F 2 "" H 1650 1450 50  0001 C CNN
+F 2 "Connector_Coaxial:SMA_Amphenol_132203-12_Horizontal" H 1650 1450 50  0001 C CNN
 F 3 "~" H 1650 1450 50  0001 C CNN
 	1    1650 1450
@@
 F 0 "J2" H 1568 1825 50  0000 C CNN
 F 1 "Conn_01x02" H 1568 1916 50  0000 C CNN
-F 2 "" H 1650 2150 50  0001 C CNN
+F 2 "Connector_Coaxial:SMA_Amphenol_132203-12_Horizontal" H 1650 2150 50  0001 C CNN
 F 3 "~" H 1650 2150 50  0001 C CNN
 	1    1650 2150
@@
 F 0 "J3" H 1568 2525 50  0000 C CNN
 F 1 "Conn_01x02" H 1568 2616 50  0000 C CNN
-F 2 "" H 1650 2850 50  0001 C CNN
+F 2 "Connector_Coaxial:SMA_Amphenol_132203-12_Horizontal" H 1650 2850 50  0001 C CNN
 F 3 "~" H 1650 2850 50  0001 C CNN
 	1    1650 2850
@@
 F 0 "J4" H 1568 3225 50  0000 C CNN
 F 1 "Conn_01x02" H 1568 3316 50  0000 C CNN
-F 2 "" H 1650 3550 50  0001 C CNN
+F 2 "Connector_Coaxial:SMA_Amphenol_132203-12_Horizontal" H 1650 3550 50  0001 C CNN
 F 3 "~" H 1650 3550 50  0001 C CNN
 	1    1650 3550
@@
 F 0 "J5" H 1568 3925 50  0000 C CNN
 F 1 "Conn_01x02" H 1568 4016 50  0000 C CNN
-F 2 "" H 1650 4250 50  0001 C CNN
+F 2 "Connector_Coaxial:SMA_Amphenol_132203-12_Horizontal" H 1650 4250 50  0001 C CNN
 F 3 "~" H 1650 4250 50  0001 C CNN
 	1    1650 4250
@@
 F 0 "J6" H 1568 4625 50  0000 C CNN
 F 1 "Conn_01x02" H 1568 4716 50  0000 C CNN
-F 2 "" H 1650 4950 50  0001 C CNN
+F 2 "Connector_Coaxial:SMA_Amphenol_132203-12_Horizontal" H 1650 4950 50  0001 C CNN
 F 3 "~" H 1650 4950 50  0001 C CNN
 	1    1650 4950
@@
 F 0 "J8" H 7530 2342 50  0000 L CNN
 F 1 "Conn_01x02" H 7530 2251 50  0000 L CNN
-F 2 "" H 7450 2350 50  0001 C CNN
+F 2 "Connector_Coaxial:SMA_Amphenol_132203-12_Horizontal" H 7450 2350 50  0001 C CNN
 F 3 "~" H 7450 2350 50  0001 C CNN
 	1    7450 2350
@@
 F 0 "J9" H 7530 3042 50  0000 L CNN
 F 1 "Conn_01x02" H 7530 2951 50  0000 L CNN
-F 2 "" H 7450 3050 50  0001 C CNN
+F 2 "Connector_Coaxial:SMA_Amphenol_132203-12_Horizontal" H 7450 3050 50  0001 C CNN
 F 3 "~" H 7450 3050 50  0001 C CNN
 	1    7450 3050
@@
 F 0 "J10" H 7530 3742 50  0000 L CNN
 F 1 "Conn_01x02" H 7530 3651 50  0000 L CNN
-F 2 "" H 7450 3750 50  0001 C CNN
+F 2 "Connector_Coaxial:SMA_Amphenol_132203-12_Horizontal" H 7450 3750 50  0001 C CNN
 F 3 "~" H 7450 3750 50  0001 C CNN
 	1    7450 3750
@@
 F 0 "J11" H 7530 4442 50  0000 L CNN
 F 1 "Conn_01x02" H 7530 4351 50  0000 L CNN
-F 2 "" H 7450 4450 50  0001 C CNN
+F 2 "Connector_Coaxial:SMA_Amphenol_132203-12_Horizontal" H 7450 4450 50  0001 C CNN
 F 3 "~" H 7450 4450 50  0001 C CNN
 	1    7450 4450
@@
 F 0 "J7" H 7530 1692 50  0000 L CNN
 F 1 "Conn_01x02" H 7530 1601 50  0000 L CNN
-F 2 "" H 7450 1700 50  0001 C CNN
+F 2 "Connector_Coaxial:SMA_Amphenol_132203-12_Horizontal" H 7450 1700 50  0001 C CNN
 F 3 "~" H 7450 1700 50  0001 C CNN
 	1    7450 1700
@@
 F 0 "J12" H 7530 5092 50  0000 L CNN
 F 1 "Conn_01x02" H 7530 5001 50  0000 L CNN
-F 2 "" H 7450 5100 50  0001 C CNN
+F 2 "Connector_Coaxial:SMA_Amphenol_132203-12_Horizontal" H 7450 5100 50  0001 C CNN
 F 3 "~" H 7450 5100 50  0001 C CNN
 	1    7450 5100

Commit message: power splitter: add LCSC part numbers
Parts:
- J1, J10, J11, J12, J2, J3, J4, J5, J6, J7, J8, J9: LCSC (none) -> C411575
- R1, R10, R11, R12, R13, R14, R15, R16, R17, R18, R19, R2, R20, R21, R22, R23, R24, R3, R4, R5, R6, R7, R8, R9: LCSC (none) -> C25136
Changed lines of the file:
@@
 F 2 "Resistor_SMD:R_0402_1005Metric" V 2980 1350 50  0001 C CNN
 F 3 "~" H 3050 1350 50  0001 C CNN
+F 4 "C25136" H 3050 1350 50  0001 C CNN "LCSC"
 	1    3050 1350
 	0    -1   -1   0
@@
 F 2 "Resistor_SMD:R_0402_1005Metric" V 2980 1650 50  0001 C CNN
 F 3 "~" H 3050 1650 50  0001 C CNN
+F 4 "C25136" H 3050 1650 50  0001 C CNN "LCSC"
 	1    3050 1650
 	0    -1   -1   0
@@
 F 2 "Resistor_SMD:R_0402_1005Metric" V 2980 2050 50  0001 C CNN
 F 3 "~" H 3050 2050 50  0001 C CNN
+F 4 "C25136" H 3050 2050 50  0001 C CNN "LCSC"
 	1    3050 2050
 	0    -1   -1   0
@@
 F 2 "Resistor_SMD:R_0402_1005Metric" V 2980 2750 50  0001 C CNN
 F 3 "~" H 3050 2750 50  0001 C CNN
+F 4 "C25136" H 3050 2750 50  0001 C CNN "LCSC"
 	1    3050 2750
 	0    -1   -1   0
@@
 F 2 "Resistor_SMD:R_0402_1005Metric" V 2980 3050 50  0001 C CNN
 F 3 "~" H 3050 3050 50  0001 C CNN
+F 4 "C25136" H 3050 3050 50  0001 C CNN "LCSC"
 	1    3050 3050
 	0    -1   -1   0
@@
 F 2 "Resistor_SMD:R_0402_1005Metric" V 2980 3450 50  0001 C CNN
 F 3 "~" H 3050 3450 50  0001 C CNN
+F 4 "C25136" H 3050 3450 50  0001 C CNN "LCSC"
 	1    3050 3450
 	0    -1   -1   0
@@
 F 2 "Resistor_SMD:R_0402_1005Metric" V 2980 3750 50  0001 C CNN
 F 3 "~" H 3050 3750 50  0001 C CNN
+F 4 "C25136" H 3050 3750 50  0001 C CNN "LCSC"
 	1    3050 3750
 	0    -1   -1   0
@@
 F 2 "Resistor_SMD:R_0402_1005Metric" V 2980 4150 50  0001 C CNN
 F 3 "~" H 3050 4150 50  0001 C CNN
+F 4 "C25136" H 3050 4150 50  0001 C CNN "LCSC"
 	1    3050 4150
 	0    -1   -1   0
@@
 F 2 "Resistor_SMD:R_0402_1005Metric" V 2980 4450 50  0001 C CNN
 F 3 "~" H 3050 4450 50  0001 C CNN
+F 4 "C25136" H 3050 4450 50  0001 C CNN "LCSC"
 	1    3050 4450
 	0    -1   -1   0
@@
 F 2 "Resistor_SMD:R_0402_1005Metric" V 2980 4850 50  0001 C CNN
 F 3 "~" H 3050 4850 50  0001 C CNN
+F 4 "C25136" H 3050 4850 50  0001 C CNN "LCSC"
 	1    3050 4850
 	0    -1   -1   0
@@
 F 2 "Resistor_SMD:R_0402_1005Metric" V 2980 5150 50  0001 C CNN
 F 3 "~" H 3050 5150 50  0001 C CNN
+F 4 "C25136" H 3050 5150 50  0001 C CNN "LCSC"
 	1    3050 5150
 	0    -1   -1   0
@@
 F 2 "Resistor_SMD:R_0402_1005Metric" V 6530 1700 50  0001 C CNN
 F 3 "~" H 6600 1700 50  0001 C CNN
+F 4 "C25136" H 6600 1700 50  0001 C CNN "LCSC"
 	1    6600 1700
 	0    -1   -1   0
@@
 F 2 "Resistor_SMD:R_0402_1005Metric" V 6530 2000 50  0001 C CNN
 F 3 "~" H 6600 2000 50  0001 C CNN
+F 4 "C25136" H 6600 2000 50  0001 C CNN "LCSC"
 	1    6600 2000
 	0    -1   -1   0
@@
 F 2 "Resistor_SMD:R_0402_1005Metric" V 6530 2350 50  0001 C CNN
 F 3 "~" H 6600 2350 50  0001 C CNN
+F 4 "C25136" H 6600 2350 50  0001 C CNN "LCSC"
 	1    6600 2350
 	0    -1   -1   0
@@
 F 2 "Resistor_SMD:R_0402_1005Metric" V 6530 2650 50  0001 C CNN
 F 3 "~" H 6600 2650 50  0001 C CNN
+F 4 "C25136" H 6600 2650 50  0001 C CNN "LCSC"
 	1    6600 2650
 	0    -1   -1   0
@@
 F 2 "Resistor_SMD:R_0402_1005Metric" V 6530 3050 50  0001 C CNN
 F 3 "~" H 6600 3050 50  0001 C CNN
+F 4 "C25136" H 6600 3050 50  0001 C CNN "LCSC"
 	1    6600 3050
 	0    -1   -1   0
@@
 F 2 "Resistor_SMD:R_0402_1005Metric" V 6530 3350 50  0001 C CNN
 F 3 "~" H 6600 3350 50  0001 C CNN
+F 4 "C25136" H 6600 3350 50  0001 C CNN "LCSC"
 	1    6600 3350
 	0    -1   -1   0
@@
 F 2 "Resistor_SMD:R_0402_1005Metric" V 6530 3750 50  0001 C CNN
 F 3 "~" H 6600 3750 50  0001 C CNN
+F 4 "C25136" H 6600 3750 50  0001 C CNN "LCSC"
 	1    6600 3750
 	0    -1   -1   0
@@
 F 2 "Resistor_SMD:R_0402_1005Metric" V 6530 4050 50  0001 C CNN
 F 3 "~" H 6600 4050 50  0001 C CNN
+F 4 "C25136" H 6600 4050 50  0001 C CNN "LCSC"
 	1    6600 4050
 	0    -1   -1   0
@@
 F 2 "Resistor_SMD:R_0402_1005Metric" V 6530 4450 50  0001 C CNN
 F 3 "~" H 6600 4450 50  0001 C CNN
+F 4 "C25136" H 6600 4450 50  0001 C CNN "LCSC"
 	1    6600 4450
 	0    -1   -1   0
@@
 F 2 "Resistor_SMD:R_0402_1005Metric" V 6530 4750 50  0001 C CNN
 F 3 "~" H 6600 4750 50  0001 C CNN
+F 4 "C25136" H 6600 4750 50  0001 C CNN "LCSC"
 	1    6600 4750
 	0    -1   -1   0
@@
 F 2 "Connector_Coaxial:SMA_Amphenol_132203-12_Horizontal" H 1650 1450 50  0001 C CNN
 F 3 "~" H 1650 1450 50  0001 C CNN
+F 4 "C411575" H 1650 1450 50  0001 C CNN "LCSC"
 	1    1650 1450
 	-1   0    0    1
@@
 F 2 "Connector_Coaxial:SMA_Amphenol_132203-12_Horizontal" H 1650 2150 50  0001 C CNN
 F 3 "~" H 1650 2150 50  0001 C CNN
+F 4 "C411575" H 1650 2150 50  0001 C CNN "LCSC"
 	1    1650 2150
 	-1   0    0    1
@@
 F 2 "Connector_Coaxial:SMA_Amphenol_132203-12_Horizontal" H 1650 2850 50  0001 C CNN
 F 3 "~" H 1650 2850 50  0001 C CNN
+F 4 "C411575" H 1650 2850 50  0001 C CNN "LCSC"
 	1    1650 2850
 	-1   0    0    1
@@
 F 2 "Connector_Coaxial:SMA_Amphenol_132203-12_Horizontal" H 1650 3550 50  0001 C CNN
 F 3 "~" H 1650 3550 50  0001 C CNN
+F 4 "C411575" H 1650 3550 50  0001 C CNN "LCSC"
 	1    1650 3550
 	-1   0    0    1
@@
 F 2 "Connector_Coaxial:SMA_Amphenol_132203-12_Horizontal" H 1650 4250 50  0001 C CNN
 F 3 "~" H 1650 4250 50  0001 C CNN
+F 4 "C411575" H 1650 4250 50  0001 C CNN "LCSC"
 	1    1650 4250
 	-1   0    0    1
@@
 F 2 "Connector_Coaxial:SMA_Amphenol_132203-12_Horizontal" H 1650 4950 50  0001 C CNN
 F 3 "~" H 1650 4950 50  0001 C CNN
+F 4 "C411575" H 1650 4950 50  0001 C CNN "LCSC"
 	1    1650 4950
 	-1   0    0    1
@@
 F 2 "Connector_Coaxial:SMA_Amphenol_132203-12_Horizontal" H 7450 2350 50  0001 C CNN
 F 3 "~" H 7450 2350 50  0001 C CNN
+F 4 "C411575" H 7450 2350 50  0001 C CNN "LCSC"
 	1    7450 2350
 	1    0    0    -1
@@
 F 2 "Connector_Coaxial:SMA_Amphenol_132203-12_Horizontal" H 7450 3050 50  0001 C CNN
 F 3 "~" H 7450 3050 50  0001 C CNN
+F 4 "C411575" H 7450 3050 50  0001 C CNN "LCSC"
 	1    7450 3050
 	1    0    0    -1
@@
 F 2 "Connector_Coaxial:SMA_Amphenol_132203-12_Horizontal" H 7450 3750 50  0001 C CNN
 F 3 "~" H 7450 3750 50  0001 C CNN
+F 4 "C411575" H 7450 3750 50  0001 C CNN "LCSC"
 	1    7450 3750
 	1    0    0    -1
@@
 F 2 "Connector_Coaxial:SMA_Amphenol_132203-12_Horizontal" H 7450 4450 50  0001 C CNN
 F 3 "~" H 7450 4450 50  0001 C CNN
+F 4 "C411575" H 7450 4450 50  0001 C CNN "LCSC"
 	1    7450 4450
 	1    0    0    -1
@@
 F 2 "Connector_Coaxial:SMA_Amphenol_132203-12_Horizontal" H 7450 1700 50  0001 C CNN
 F 3 "~" H 7450 1700 50  0001 C CNN
+F 4 "C411575" H 7450 1700 50  0001 C CNN "LCSC"
 	1    7450 1700
 	1    0    0    -1
@@
 F 2 "Resistor_SMD:R_0402_1005Metric" V 2980 2350 50  0001 C CNN
 F 3 "~" H 3050 2350 50  0001 C CNN
+F 4 "C25136" H 3050 2350 50  0001 C CNN "LCSC"
 	1    3050 2350
 	0    -1   -1   0
@@
 F 2 "Resistor_SMD:R_0402_1005Metric" V 6530 5100 50  0001 C CNN
 F 3 "~" H 6600 5100 50  0001 C CNN
+F 4 "C25136" H 6600 5100 50  0001 C CNN "LCSC"
 	1    6600 5100
 	0    -1   -1   0
@@
 F 2 "Resistor_SMD:R_0402_1005Metric" V 6530 5400 50  0001 C CNN
 F 3 "~" H 6600 5400 50  0001 C CNN
+F 4 "C25136" H 6600 5400 50  0001 C CNN "LCSC"
 	1    6600 5400
 	0    -1   -1   0
@@
 F 2 "Connector_Coaxial:SMA_Amphenol_132203-12_Horizontal" H 7450 5100 50  0001 C CNN
 F 3 "~" H 7450 5100 50  0001 C CNN
+F 4 "C411575" H 7450 5100 50  0001 C CNN "LCSC"
 	1    7450 5100
 	1    0    0    -1

Commit message: power splitter: add footprint field to schematic
Parts:
- R1, R10, R11, R12, R13, R14, R15, R16, R17, R18, R19, R2, R20, R21, R22, R23, R24, R3, R4, R5, R6, R7, R8, R9: JLC (none) -> 0402
Changed lines of the file:
@@
 F 3 "~" H 3050 1350 50  0001 C CNN
 F 4 "C25136" H 3050 1350 50  0001 C CNN "LCSC"
+F 5 "0402" H 3050 1350 50  0001 C CNN "JLC"
 	1    3050 1350
 	0    -1   -1   0
@@
 F 3 "~" H 3050 1650 50  0001 C CNN
 F 4 "C25136" H 3050 1650 50  0001 C CNN "LCSC"
+F 5 "0402" H 3050 1650 50  0001 C CNN "JLC"
 	1    3050 1650
 	0    -1   -1   0
@@
 F 3 "~" H 3050 2050 50  0001 C CNN
 F 4 "C25136" H 3050 2050 50  0001 C CNN "LCSC"
+F 5 "0402" H 3050 2050 50  0001 C CNN "JLC"
 	1    3050 2050
 	0    -1   -1   0
@@
 F 3 "~" H 3050 2750 50  0001 C CNN
 F 4 "C25136" H 3050 2750 50  0001 C CNN "LCSC"
+F 5 "0402" H 3050 2750 50  0001 C CNN "JLC"
 	1    3050 2750
 	0    -1   -1   0
@@
 F 3 "~" H 3050 3050 50  0001 C CNN
 F 4 "C25136" H 3050 3050 50  0001 C CNN "LCSC"
+F 5 "0402" H 3050 3050 50  0001 C CNN "JLC"
 	1    3050 3050
 	0    -1   -1   0
@@
 F 3 "~" H 3050 3450 50  0001 C CNN
 F 4 "C25136" H 3050 3450 50  0001 C CNN "LCSC"
+F 5 "0402" H 3050 3450 50  0001 C CNN "JLC"
 	1    3050 3450
 	0    -1   -1   0
@@
 F 3 "~" H 3050 3750 50  0001 C CNN
 F 4 "C25136" H 3050 3750 50  0001 C CNN "LCSC"
+F 5 "0402" H 3050 3750 50  0001 C CNN "JLC"
 	1    3050 3750
 	0    -1   -1   0
@@
 F 3 "~" H 3050 4150 50  0001 C CNN
 F 4 "C25136" H 3050 4150 50  0001 C CNN "LCSC"
+F 5 "0402" H 3050 4150 50  0001 C CNN "JLC"
 	1    3050 4150
 	0    -1   -1   0
@@
 F 3 "~" H 3050 4450 50  0001 C CNN
 F 4 "C25136" H 3050 4450 50  0001 C CNN "LCSC"
+F 5 "0402" H 3050 4450 50  0001 C CNN "JLC"
 	1    3050 4450
 	0    -1   -1   0
@@
 F 3 "~" H 3050 4850 50  0001 C CNN
 F 4 "C25136" H 3050 4850 50  0001 C CNN "LCSC"
+F 5 "0402" H 3050 4850 50  0001 C CNN "JLC"
 	1    3050 4850
 	0    -1   -1   0
@@
 F 3 "~" H 3050 5150 50  0001 C CNN
 F 4 "C25136" H 3050 5150 50  0001 C CNN "LCSC"
+F 5 "0402" H 3050 5150 50  0001 C CNN "JLC"
 	1    3050 5150
 	0    -1   -1   0
@@
 F 3 "~" H 6600 1700 50  0001 C CNN
 F 4 "C25136" H 6600 1700 50  0001 C CNN "LCSC"
+F 5 "0402" H 6600 1700 50  0001 C CNN "JLC"
 	1    6600 1700
 	0    -1   -1   0
@@
 F 3 "~" H 6600 2000 50  0001 C CNN
 F 4 "C25136" H 6600 2000 50  0001 C CNN "LCSC"
+F 5 "0402" H 6600 2000 50  0001 C CNN "JLC"
 	1    6600 2000
 	0    -1   -1   0
@@
 F 3 "~" H 6600 2350 50  0001 C CNN
 F 4 "C25136" H 6600 2350 50  0001 C CNN "LCSC"
+F 5 "0402" H 6600 2350 50  0001 C CNN "JLC"
 	1    6600 2350
 	0    -1   -1   0
@@
 F 3 "~" H 6600 2650 50  0001 C CNN
 F 4 "C25136" H 6600 2650 50  0001 C CNN "LCSC"
+F 5 "0402" H 6600 2650 50  0001 C CNN "JLC"
 	1    6600 2650
 	0    -1   -1   0
@@
 F 3 "~" H 6600 3050 50  0001 C CNN
 F 4 "C25136" H 6600 3050 50  0001 C CNN "LCSC"
+F 5 "0402" H 6600 3050 50  0001 C CNN "JLC"
 	1    6600 3050
 	0    -1   -1   0
@@
 F 3 "~" H 6600 3350 50  0001 C CNN
 F 4 "C25136" H 6600 3350 50  0001 C CNN "LCSC"
+F 5 "0402" H 6600 3350 50  0001 C CNN "JLC"
 	1    6600 3350
 	0    -1   -1   0
@@
 F 3 "~" H 6600 3750 50  0001 C CNN
 F 4 "C25136" H 6600 3750 50  0001 C CNN "LCSC"
+F 5 "0402" H 6600 3750 50  0001 C CNN "JLC"
 	1    6600 3750
 	0    -1   -1   0
@@
 F 3 "~" H 6600 4050 50  0001 C CNN
 F 4 "C25136" H 6600 4050 50  0001 C CNN "LCSC"
+F 5 "0402" H 6600 4050 50  0001 C CNN "JLC"
 	1    6600 4050
 	0    -1   -1   0
@@
 F 3 "~" H 6600 4450 50  0001 C CNN
 F 4 "C25136" H 6600 4450 50  0001 C CNN "LCSC"
+F 5 "0402" H 6600 4450 50  0001 C CNN "JLC"
 	1    6600 4450
 	0    -1   -1   0
@@
 F 3 "~" H 6600 4750 50  0001 C CNN
 F 4 "C25136" H 6600 4750 50  0001 C CNN "LCSC"
+F 5 "0402" H 6600 4750 50  0001 C CNN "JLC"
 	1    6600 4750
 	0    -1   -1   0
@@
 F 3 "~" H 3050 2350 50  0001 C CNN
 F 4 "C25136" H 3050 2350 50  0001 C CNN "LCSC"
+F 5 "0402" H 3050 2350 50  0001 C CNN "JLC"
 	1    3050 2350
 	0    -1   -1   0
@@
 F 3 "~" H 6600 5100 50  0001 C CNN
 F 4 "C25136" H 6600 5100 50  0001 C CNN "LCSC"
+F 5 "0402" H 6600 5100 50  0001 C CNN "JLC"
 	1    6600 5100
 	0    -1   -1   0
@@
 F 3 "~" H 6600 5400 50  0001 C CNN
 F 4 "C25136" H 6600 5400 50  0001 C CNN "LCSC"
+F 5 "0402" H 6600 5400 50  0001 C CNN "JLC"
 	1    6600 5400
 	0    -1   -1   0
