File: power_splitter/resistive-power-splitter.kicad_pcb (KiCad board)
At the start: 4 copper layers, 58 x 58 mm, 24 parts, among them J1 Conn_01x02, J10 Conn_01x02, J11 Conn_01x02, J12 Conn_01x02, J2 Conn_01x02, J3 Conn_01x02, J4 Conn_01x02, J5 Conn_01x02, J6 Conn_01x02, J7 Conn_01x02, J8 Conn_01x02, J9 Conn_01x02

Commit message: power splitter: use custom footprint with associated 3d model for SMA connectors
Parts:
- J1, J10, J11, J12, J2, J3, J4, J5, J6, J7, J8, J9: footprint Connector_Coaxial:SMA_Amphenol_132203-12_Horizontal -> custom_library:SMA_HJ-SMA003

Commit message: power splitter: adjust footprint info of SMA connector
The v2 model of the SMA connector no longer requires the Z-offset of 0.5
mm.

Note: this also converts the PCB to KiCad 6.0.
Other:
- net class Default removed
