File: lemonbeat_dongle/mcu.kicad_sch (KiCad schematic)
At the start: 44 parts, among them J201 USB_A, J202 Prog, J203 u.FL, SW201 SW_Push, U201 nRF52840, Y201 32MHz, Y202 32.768kHz

Commit message: dongle: use capacitor footprints for capacitors
(rather than identical resistor footprints)
Parts:
- C201, C202, C203, C204, C205, C206, C208, C209, C210, C211, C212, C214, C216, C217, C218, C222, C223, C224, C225, C226: footprint Resistor_SMD:R_0201_0603Metric -> Capacitor_SMD:C_0201_0603Metric
- C207, C215: footprint Resistor_SMD:R_0402_1005Metric -> Capacitor_SMD:C_0402_1005Metric
- C213, C219, C220, C221: footprint Resistor_SMD:R_0603_1608Metric -> Capacitor_SMD:C_0603_1608Metric
Changed lines of the file:
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@@
       (effects (font (size 1.27 1.27)) (justify left))
     )
-    (property "Footprint" "Resistor_SMD:R_0201_0603Metric" (id 2) (at 32.7152 171.45 0)
+    (property "Footprint" "Capacitor_SMD:C_0201_0603Metric" (id 2) (at 32.7152 171.45 0)
       (effects (font (size 1.27 1.27)) hide)
     )
@@
       (effects (font (size 1.27 1.27)) (justify left))
     )
-    (property "Footprint" "Resistor_SMD:R_0402_1005Metric" (id 2) (at 70.8152 30.48 0)
+    (property "Footprint" "Capacitor_SMD:C_0402_1005Metric" (id 2) (at 70.8152 30.48 0)
       (effects (font (size 1.27 1.27)) hide)
     )
@@
       (effects (font (size 1.27 1.27)) (justify left))
     )
-    (property "Footprint" "Resistor_SMD:R_0201_0603Metric" (id 2) (at 163.5252 27.94 0)
+    (property "Footprint" "Capacitor_SMD:C_0201_0603Metric" (id 2) (at 163.5252 27.94 0)
       (effects (font (size 1.27 1.27)) hide)
     )
@@
       (effects (font (size 1.27 1.27)) (justify left))
     )
-    (property "Footprint" "Resistor_SMD:R_0201_0603Metric" (id 2) (at 178.7652 138.43 0)
+    (property "Footprint" "Capacitor_SMD:C_0201_0603Metric" (id 2) (at 178.7652 138.43 0)
       (effects (font (size 1.27 1.27)) hide)
     )
@@
       (effects (font (size 1.27 1.27)) (justify right))
     )
-    (property "Footprint" "Resistor_SMD:R_0603_1608Metric" (id 2) (at 18.0848 83.82 0)
+    (property "Footprint" "Capacitor_SMD:C_0603_1608Metric" (id 2) (at 18.0848 83.82 0)
       (effects (font (size 1.27 1.27)) hide)
     )
@@
       (effects (font (size 1.27 1.27)) (justify left))
     )
-    (property "Footprint" "Resistor_SMD:R_0201_0603Metric" (id 2) (at 237.1852 60.96 0)
+    (property "Footprint" "Capacitor_SMD:C_0201_0603Metric" (id 2) (at 237.1852 60.96 0)
       (effects (font (size 1.27 1.27)) hide)
     )
@@
       (effects (font (size 1.27 1.27)) (justify left))
     )
-    (property "Footprint" "Resistor_SMD:R_0201_0603Metric" (id 2) (at 50.4952 48.26 0)
+    (property "Footprint" "Capacitor_SMD:C_0201_0603Metric" (id 2) (at 50.4952 48.26 0)
       (effects (font (size 1.27 1.27)) hide)
     )
@@
       (effects (font (size 1.27 1.27)) (justify left))
     )
-    (property "Footprint" "Resistor_SMD:R_0201_0603Metric" (id 2) (at 113.9952 27.94 0)
+    (property "Footprint" "Capacitor_SMD:C_0201_0603Metric" (id 2) (at 113.9952 27.94 0)
       (effects (font (size 1.27 1.27)) hide)
     )
@@
       (effects (font (size 1.27 1.27)) (justify left))
     )
-    (property "Footprint" "Resistor_SMD:R_0201_0603Metric" (id 2) (at 28.9052 71.12 0)
+    (property "Footprint" "Capacitor_SMD:C_0201_0603Metric" (id 2) (at 28.9052 71.12 0)
       (effects (font (size 1.27 1.27)) hide)
     )
@@
     (property "Reference" "C204" (id 0) (at 151.13 57.15 90))
     (property "Value" "12pF" (id 1) (at 151.13 64.77 90))
-    (property "Footprint" "Resistor_SMD:R_0201_0603Metric" (id 2) (at 154.94 59.9948 0)
+    (property "Footprint" "Capacitor_SMD:C_0201_0603Metric" (id 2) (at 154.94 59.9948 0)
       (effects (font (size 1.27 1.27)) hide)
     )
@@
       (effects (font (size 1.27 1.27)) (justify left))
     )
-    (property "Footprint" "Resistor_SMD:R_0201_0603Metric" (id 2) (at 224.4852 60.96 0)
+    (property "Footprint" "Capacitor_SMD:C_0201_0603Metric" (id 2) (at 224.4852 60.96 0)
       (effects (font (size 1.27 1.27)) hide)
     )
@@
       (effects (font (size 1.27 1.27)) (justify left))
     )
-    (property "Footprint" "Resistor_SMD:R_0201_0603Metric" (id 2) (at 16.2052 48.26 0)
+    (property "Footprint" "Capacitor_SMD:C_0201_0603Metric" (id 2) (at 16.2052 48.26 0)
       (effects (font (size 1.27 1.27)) hide)
     )
@@
       (effects (font (size 1.27 1.27)) (justify left))
     )
-    (property "Footprint" "Resistor_SMD:R_0201_0603Metric" (id 2) (at 188.9252 138.43 0)
+    (property "Footprint" "Capacitor_SMD:C_0201_0603Metric" (id 2) (at 188.9252 138.43 0)
       (effects (font (size 1.27 1.27)) hide)
     )
@@
     (property "Reference" "C202" (id 0) (at 27.94 116.84 90))
     (property "Value" "12pF" (id 1) (at 27.94 119.38 90))
-    (property "Footprint" "Resistor_SMD:R_0201_0603Metric" (id 2) (at 31.75 122.2248 0)
+    (property "Footprint" "Capacitor_SMD:C_0201_0603Metric" (id 2) (at 31.75 122.2248 0)
       (effects (font (size 1.27 1.27)) hide)
     )
@@
     (property "Reference" "C203" (id 0) (at 151.13 46.99 90))
     (property "Value" "12pF" (id 1) (at 151.13 54.61 90))
-    (property "Footprint" "Resistor_SMD:R_0201_0603Metric" (id 2) (at 147.32 51.7652 0)
+    (property "Footprint" "Capacitor_SMD:C_0201_0603Metric" (id 2) (at 147.32 51.7652 0)
       (effects (font (size 1.27 1.27)) hide)
     )
@@
       (effects (font (size 1.27 1.27)) (justify left))
     )
-    (property "Footprint" "Resistor_SMD:R_0603_1608Metric" (id 2) (at 18.7452 71.12 0)
+    (property "Footprint" "Capacitor_SMD:C_0603_1608Metric" (id 2) (at 18.7452 71.12 0)
       (effects (font (size 1.27 1.27)) hide)
     )
@@
       (effects (font (size 1.27 1.27)) (justify left))
     )
-    (property "Footprint" "Resistor_SMD:R_0201_0603Metric" (id 2) (at 252.4252 96.52 0)
+    (property "Footprint" "Capacitor_SMD:C_0201_0603Metric" (id 2) (at 252.4252 96.52 0)
       (effects (font (size 1.27 1.27)) hide)
     )
@@
       (effects (font (size 1.27 1.27)) (justify left))
     )
-    (property "Footprint" "Resistor_SMD:R_0402_1005Metric" (id 2) (at 216.8652 60.96 0)
+    (property "Footprint" "Capacitor_SMD:C_0402_1005Metric" (id 2) (at 216.8652 60.96 0)
       (effects (font (size 1.27 1.27)) hide)
     )
@@
       (effects (font (size 1.27 1.27)) (justify left))
     )
-    (property "Footprint" "Resistor_SMD:R_0603_1608Metric" (id 2) (at 139.3952 27.94 0)
+    (property "Footprint" "Capacitor_SMD:C_0603_1608Metric" (id 2) (at 139.3952 27.94 0)
       (effects (font (size 1.27 1.27)) hide)
     )
@@
       (effects (font (size 1.27 1.27)) (justify left))
     )
-    (property "Footprint" "Resistor_SMD:R_0201_0603Metric" (id 2) (at 102.5652 27.94 0)
+    (property "Footprint" "Capacitor_SMD:C_0201_0603Metric" (id 2) (at 102.5652 27.94 0)
       (effects (font (size 1.27 1.27)) hide)
     )
@@
       (effects (font (size 1.27 1.27)) (justify left))
     )
-    (property "Footprint" "Resistor_SMD:R_0201_0603Metric" (id 2) (at 168.6052 138.43 0)
+    (property "Footprint" "Capacitor_SMD:C_0201_0603Metric" (id 2) (at 168.6052 138.43 0)
       (effects (font (size 1.27 1.27)) hide)
     )
@@
       (effects (font (size 1.27 1.27)) (justify left))
     )
-    (property "Footprint" "Resistor_SMD:R_0201_0603Metric" (id 2) (at 125.4252 27.94 0)
+    (property "Footprint" "Capacitor_SMD:C_0201_0603Metric" (id 2) (at 125.4252 27.94 0)
       (effects (font (size 1.27 1.27)) hide)
     )
@@
     (property "Reference" "C201" (id 0) (at 27.94 106.68 90))
     (property "Value" "12pF" (id 1) (at 27.94 109.22 90))
-    (property "Footprint" "Resistor_SMD:R_0201_0603Metric" (id 2) (at 31.75 112.0648 0)
+    (property "Footprint" "Capacitor_SMD:C_0201_0603Metric" (id 2) (at 31.75 112.0648 0)
       (effects (font (size 1.27 1.27)) hide)
     )
@@
       (effects (font (size 1.27 1.27)) (justify left))
     )
-    (property "Footprint" "Resistor_SMD:R_0603_1608Metric" (id 2) (at 150.8252 27.94 0)
+    (property "Footprint" "Capacitor_SMD:C_0603_1608Metric" (id 2) (at 150.8252 27.94 0)
       (effects (font (size 1.27 1.27)) hide)
     )
@@
       (effects (font (size 1.27 1.27)) (justify left))
     )
-    (property "Footprint" "Resistor_SMD:R_0201_0603Metric" (id 2) (at 26.3652 48.26 0)
+    (property "Footprint" "Capacitor_SMD:C_0201_0603Metric" (id 2) (at 26.3652 48.26 0)
       (effects (font (size 1.27 1.27)) hide)
     )
@@
       (effects (font (size 1.27 1.27)) (justify left))
     )
-    (property "Footprint" "Resistor_SMD:R_0201_0603Metric" (id 2) (at 36.5252 48.26 0)
-      (effects (font (size 1.27 1.27)) hide)
-    )
+    (property "Footprint" "Capacitor_SMD:C_0201_0603Metric" (id 2) (at 36.5252 48.26 0)
+      (effects (font (size 1.27 1.27)) hide)
+    )
