File: lemonbeat_dongle/dongle.kicad_sch (KiCad schematic)
At the start: 6 parts

Commit message: dongle: update date & revision; typo fix
Other:
- title: BNW Lemonbeat Donlge -> BNW Lemonbeat Dongle
Changed lines of the file:
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@@
   (paper "A4")
   (title_block
-    (title "BNW Lemonbeat Donlge")
-    (date "21.10.2022")
-    (rev "0.2.0")
+    (title "BNW Lemonbeat Dongle")
+    (date "10.3.2023")
+    (rev "0.3.0")
   )
   (junction (at 125.73 114.3) (diameter 0) (color 0 0 0 0)
