File: lemonbeat_dongle/transceiver.kicad_sch (KiCad schematic)
At the start: 25 parts, among them J301 SMA, U301 Si4467, Y301 26MHz

Commit message: dongle: replace parts not available at JLCPCB
These parts were all unavailable for rev. 0.3.0 and are still
unavailable.

Replacements:
- FB201, FB202: C281196 -> C2662025 (same replacement as for rev. 0.3.0)
- J203: C88373 -> C598199 (same replacement as for rev. 0.3.0; this
  seems to be only a packaging change)
- L301: C335569 -> C86067 (rev. 0.2.0 and 0.3.0 uses C268315, but C86067
  is from Murata, has lower DC resistance and slightly better current
  rating)
- L303: C87185 -> C84404 (rev. 0.3.0 uses C237609, but C84404 has better
  tolerance)
- L305, L306: C335566 -> C882467 (rev. 0.2.0 and 0.3.0 used C96056 as
  replacement, but C882467 has lower tolerance and better current
  rating)
- R203: C247442 -> C3152027 (same replacement as for rev. 0.3.0)
Parts:
- L301: Comment (none) -> Si4467 board uses CoilcCraft 0402HPH-R12XJL with 5% toleran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; LCSC C335569 -> C86067; Manufacturer Coilcraft -> Murata Electronics; Part Number 0402DC-R12XGRW -> LQG15HSR12J02D
- L303: Comment (none) -> Si4467 board uses CoilCraft 0402HP-8N2XJL with 5% tolerance.; LCSC C87185 -> C84404; Manufacturer Taiyo Yuden -> Murata Electronics; Part Number HK10058N2J-T -> LQW15AN8N2G00D
- L305, L306: Comment (none) -> Si4467 board uses CoilCraft 0402HP-6N8XJL with 5% tolerance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; LCSC C335566 -> C882467; Manufacturer Coilcraft -> Murata Electronics; Part Number 0402DC-6N8XGRW -> LQW15AN6N8G80D
Changed lines of the file:
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@@
 			)
 		)
-		(property "Datasheet" "~"
+		(property "Datasheet" "https://wmsc.lcsc.com/wmsc/upload/file/pdf/v2/lcsc/2201242130_Murata-Electronics-LQW15AN6N8G80D_C882467.pdf"
 			(at 151.13 88.9 0)
 			(effects
@@
 			)
 		)
-		(property "Description" "1.5A 6.8nH ±2% 63mΩ 0402"
+		(property "Description" "1.45A 6.8nH ±2% 0402 Power Inductors ROHS"
 			(at 151.13 88.9 0)
 			(effects
@@
 			)
 		)
-		(property "LCSC" "C335566"
+		(property "LCSC" "C882467"
 			(at 151.13 88.9 0)
 			(effects
@@
 			)
 		)
-		(property "Manufacturer" "Coilcraft"
+		(property "Manufacturer" "Murata Electronics"
 			(at 151.13 88.9 0)
 			(effects
@@
 			)
 		)
-		(property "Part Number" "0402DC-6N8XGRW"
+		(property "Part Number" "LQW15AN6N8G80D"
+			(at 151.13 88.9 0)
+			(effects
+				(font
+					(size 1.27 1.27)
+				)
+				(hide yes)
+			)
+		)
+		(property "Comment" "Si4467 board uses CoilCraft 0402HP-6N8XJL with 5% tolerance and 1500 mA current rating."
 			(at 151.13 88.9 0)
 			(effects
@@
 			)
 		)
-		(property "Datasheet" "~"
+		(property "Datasheet" "https://wmsc.lcsc.com/wmsc/upload/file/pdf/v2/lcsc/1811081516_Murata-Electronics-LQW15AN8N2G00D_C84404.pdf"
 			(at 115.57 88.9 0)
 			(effects
@@
 			)
 		)
-		(property "Description" "8.2nH ±5% 380mA 280mΩ 0402 HF Inductors"
+		(property "Description" "540mA 8.2nH ±2% 0402 Power Inductors ROHS"
 			(at 115.57 88.9 0)
 			(effects
@@
 			)
 		)
-		(property "LCSC" "C87185"
+		(property "LCSC" "C84404"
 			(at 115.57 88.9 0)
 			(effects
@@
 			)
 		)
-		(property "Manufacturer" "Taiyo Yuden"
+		(property "Manufacturer" "Murata Electronics"
 			(at 115.57 88.9 0)
 			(effects
@@
 			)
 		)
-		(property "Part Number" "HK10058N2J-T"
+		(property "Part Number" "LQW15AN8N2G00D"
 			(at 115.57 88.9 0)
+			(effects
+				(font
+					(size 1.27 1.27)
+				)
+				(hide yes)
+			)
+		)
+		(property "Comment" "Si4467 board uses CoilCraft 0402HP-8N2XJL with 5% tolerance."
+			(at 115.57 88.9 90)
 			(effects
 				(font
@@
 			)
 		)
-		(property "Datasheet" "~"
+		(property "Datasheet" "https://wmsc.lcsc.com/wmsc/upload/file/pdf/v2/lcsc/1811081614_Murata-Electronics-LQG15HSR12J02D_C86067.pdf"
 			(at 106.68 81.28 0)
 			(effects
@@
 			)
 		)
-		(property "Description" "310mA 120nH ±2% 1.6Ω 0402"
+		(property "Description" "200mA 120nH ±5% 1.3Ω 0402 Inductors (SMD)"
 			(at 106.68 81.28 0)
 			(effects
@@
 			)
 		)
-		(property "LCSC" "C335569"
+		(property "LCSC" "C86067"
 			(at 106.68 81.28 0)
 			(effects
@@
 			)
 		)
-		(property "Manufacturer" "Coilcraft"
+		(property "Manufacturer" "Murata Electronics"
 			(at 106.68 81.28 0)
 			(effects
@@
 			)
 		)
-		(property "Part Number" "0402DC-R12XGRW"
+		(property "Part Number" "LQG15HSR12J02D"
+			(at 106.68 81.28 0)
+			(effects
+				(font
+					(size 1.27 1.27)
+				)
+				(hide yes)
+			)
+		)
+		(property "Comment" "Si4467 board uses CoilcCraft 0402HPH-R12XJL with 5% tolerance, 310 mA current rating and 1.2Ω DCR."
 			(at 106.68 81.28 0)
 			(effects
@@
 			)
 		)
-		(property "Datasheet" "~"
+		(property "Datasheet" "https://wmsc.lcsc.com/wmsc/upload/file/pdf/v2/lcsc/2201242130_Murata-Electronics-LQW15AN6N8G80D_C882467.pdf"
 			(at 138.43 88.9 0)
 			(effects
@@
 			)
 		)
-		(property "Description" "1.5A 6.8nH ±2% 63mΩ 0402"
+		(property "Description" "1.45A 6.8nH ±2% 0402 Power Inductors ROHS"
 			(at 138.43 88.9 0)
 			(effects
@@
 			)
 		)
-		(property "LCSC" "C335566"
+		(property "LCSC" "C882467"
 			(at 138.43 88.9 0)
 			(effects
@@
 			)
 		)
-		(property "Manufacturer" "Coilcraft"
+		(property "Manufacturer" "Murata Electronics"
 			(at 138.43 88.9 0)
 			(effects
@@
 			)
 		)
-		(property "Part Number" "0402DC-6N8XGRW"
+		(property "Part Number" "LQW15AN6N8G80D"
 			(at 138.43 88.9 0)
 			(effects
+				(font
+					(size 1.27 1.27)
+				)
+				(hide yes)
+			)
+		)
+		(property "Comment" "Si4467 board uses CoilCraft 0402HP-6N8XJL with 5% tolerance and 1500 mA current rating."
+			(at 138.43 88.9 0)
+			(effects

Commit message: dongle: BOM: reflect manufacturing changes
Changes due to currently unavailable stock at JLCPCB:
- J203: C598199 -> C88374 (same u.FL connector in different packaging)
- C307: C723324 -> C237514 (very similar capacitor from Murata)
Parts:
- C307: LCSC C723324 -> C237514; Part Number GJM0335C1H1R0WB01D -> GJM0335C1H1R0BB01D
Changed lines of the file:
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@@
 			)
 		)
-		(property "Datasheet" "~"
+		(property "Datasheet" "https://wmsc.lcsc.com/wmsc/upload/file/pdf/v2/lcsc/1912111437_Murata-Electronics-GJM0335C1H1R0BB01D_C237514.pdf"
 			(at 119.38 27.94 0)
 			(effects
@@
 			)
 		)
-		(property "Description" "50V 1pF C0G ±0.05pF 0201"
+		(property "Description" "50V 1pF C0G 0201 MLCC"
 			(at 119.38 27.94 0)
 			(effects
@@
 			)
 		)
-		(property "LCSC" "C723324"
+		(property "LCSC" "C237514"
 			(at 119.38 27.94 0)
 			(effects
@@
 			)
 		)
-		(property "Part Number" "GJM0335C1H1R0WB01D"
+		(property "Part Number" "GJM0335C1H1R0BB01D"
 			(at 119.38 27.94 0)
 			(effects

Commit message: dongle: BOM: update C310 JLCPCB part number
C161369 -> C237422

The previous model is no longer on stock at JLCPCB and Murata GJM series
is preferable to GRM for HF circuit due to higher Q factor.
Parts:
- C310: LCSC C161369 -> C237422; Part Number GRM0335C1E100GA01D -> GJM0335C1E100GB01D
Changed lines of the file:
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@@
 			)
 		)
-		(property "Datasheet" "~"
+		(property "Datasheet" "https://wmsc.lcsc.com/wmsc/upload/file/pdf/v2/lcsc/1912111437_Murata-Electronics-GJM0335C1E100GB01D_C237422.pdf"
 			(at 144.78 96.52 0)
 			(effects
@@
 			)
 		)
-		(property "Description" "25V 10pF C0G ±2% 0201"
+		(property "Description" "25V 10pF C0G ±2% 0201 MLCC"
 			(at 144.78 96.52 0)
 			(effects
@@
 			)
 		)
-		(property "LCSC" "C161369"
+		(property "LCSC" "C237422"
 			(at 144.78 96.52 0)
 			(effects
@@
 			)
 		)
-		(property "Part Number" "GRM0335C1E100GA01D"
+		(property "Part Number" "GJM0335C1E100GB01D"
 			(at 144.78 96.52 0)
 			(effects

Commit message: dongle: BOM: C305: replace Murata GRM with GJM part
C161388 -> C701301 (GRM0335C1E3R0CA01D -> GJM0335C1E3R0CB01D)

Murata GJM series is preferable to GRM for HF circuit due to higher Q
factor.
Parts:
- C305: LCSC C161388 -> C701301; Part Number GRM0335C1E3R0CA01D -> GJM0335C1E3R0CB01D
Changed lines of the file:
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@@
 			)
 		)
-		(property "Datasheet" "~"
+		(property "Datasheet" "https://wmsc.lcsc.com/wmsc/upload/file/pdf/v2/lcsc/2201131100_Murata-Electronics-GJM0335C1E3R0CB01D_C701301.pdf"
 			(at 113.03 46.99 0)
 			(effects
@@
 			)
 		)
-		(property "LCSC" "C161388"
+		(property "LCSC" "C701301"
 			(at 113.03 46.99 0)
 			(effects
@@
 			)
 		)
-		(property "Part Number" "GRM0335C1E3R0CA01D"
+		(property "Part Number" "GJM0335C1E3R0CB01D"
 			(at 113.03 46.99 0)
 			(effects
