File: wor_dk/transceiver.kicad_sch (KiCad schematic)
At the start: 23 parts, among them J301 SMA, J302 Conn_02x04_Odd_Even, J303 Conn_02x06_Odd_Even, U301 Si4467, Y301 26MHz

Commit message: wor_dk: add all footprints & part info for connectors
Parts:
- J301: MPN (none) -> 142-0701-851; Manufacturer Johnson -> Johnson / Cinch Connectivity Solutions
- J302: LCSC (none) -> C492421; MPN (none) -> PZ254V-12-8P/; Manufacturer (none) -> XFCN
- J303: LCSC (none) -> C225521; MPN (none) -> A2541WV-2x6P; Manufacturer (none) -> CJT(Changjiang Connectors)
Changed lines of the file:
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@@
 			)
 		)
-		(property "Datasheet" "~"
+		(property "Datasheet" "https://wmsc.lcsc.com/wmsc/upload/file/pdf/v2/lcsc/2211171530_CJT-Changjiang-Connectors-A2541WV-2x6P_C225521.pdf"
 			(at 254 81.28 0)
 			(effects
@@
 		)
 		(property "Description" "Generic connector, double row, 02x06, odd/even pin numbering scheme (row 1 odd numbers, row 2 even numbers), script generated (kicad-library-utils/schlib/autogen/connector/)"
+			(at 254 81.28 0)
+			(effects
+				(font
+					(size 1.27 1.27)
+				)
+				(hide yes)
+			)
+		)
+		(property "LCSC" "C225521"
+			(at 254 81.28 0)
+			(effects
+				(font
+					(size 1.27 1.27)
+				)
+				(hide yes)
+			)
+		)
+		(property "MPN" "A2541WV-2x6P"
+			(at 254 81.28 0)
+			(effects
+				(font
+					(size 1.27 1.27)
+				)
+				(hide yes)
+			)
+		)
+		(property "Manufacturer" "CJT(Changjiang Connectors)"
 			(at 254 81.28 0)
 			(effects
@@
 			)
 		)
-		(property "Manufacturer" "Johnson"
+		(property "Manufacturer" "Johnson / Cinch Connectivity Solutions"
 			(at 217.17 93.98 0)
 			(effects
@@
 		)
 		(property "Comment" "Alternative suitable part: Amphenol RF 901-10309"
+			(at 217.17 93.98 0)
+			(effects
+				(font
+					(size 1.27 1.27)
+				)
+				(hide yes)
+			)
+		)
+		(property "MPN" "142-0701-851"
 			(at 217.17 93.98 0)
 			(effects
@@
 			)
 		)
-		(property "Datasheet" "~"
+		(property "Datasheet" "https://wmsc.lcsc.com/wmsc/upload/file/pdf/v2/lcsc/2003191006_XFCN-PZ254V-12-8P_C492421.pdf"
 			(at 254 39.37 0)
 			(effects
@@
 			(at 254 39.37 0)
 			(effects
+				(font
+					(size 1.27 1.27)
+				)
+				(hide yes)
+			)
+		)
+		(property "LCSC" "C492421"
+			(at 254 39.37 0)
+			(effects
+				(font
+					(size 1.27 1.27)
+				)
+				(hide yes)
+			)
+		)
+		(property "MPN" "PZ254V-12-8P/"
+			(at 254 39.37 0)
+			(effects
+				(font
+					(size 1.27 1.27)
+				)
+				(hide yes)
+			)
+		)
+		(property "Manufacturer" "XFCN"
+			(at 254 39.37 0)
+			(effects
