File: lemonbeat_dongle_microjig/lemonbeat_dongle_microjig.kicad_sch (KiCad schematic)
At the start: 20 parts, among them J1 Prog, J2 Main, J3 Si4467

Commit message: dongle: microjig: update to use new pogo pins
Parts:
- TP1, TP2, TP201, TP202, TP203, TP204, TP205, TP206, TP207, TP3, TP4: footprint TestPoint:TestPoint_Pad_D2.0mm -> Connector_PogoPin:PogoPin_D0.6mm_L8.4mm_W2.0mm; JLCPCB Alternatives C530675: 4mm total height; C530676: 6.5mm total height; C53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 -> Identical: C5157271; LCSC C530675 -> C5157270
- TP101, TP102, TP103, TP104, TP105, TP106: value TestPoint_Small -> TestPoint; footprint TestPoint:TestPoint_Pad_D2.0mm -> Connector_PogoPin:PogoPin_D0.6mm_L8.4mm_W2.0mm; JLCPCB Alternatives C530675: 4mm total height; C530676: 6.5mm total height; C53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 -> Identical: C5157271; LCSC C530675 -> C5157270

Commit message: dongle & micro jig: update revision to 0.4.1
Other:
- title: BNW Lemonbeat Donlge -> BNW Lemonbeat Dongle MicroJig
Changed lines of the file:
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@@
 	(paper "A4")
 	(title_block
-		(title "BNW Lemonbeat Donlge")
-		(date "22.9.2023")
-		(rev "0.4.0")
+		(title "BNW Lemonbeat Dongle MicroJig")
+		(date "25.6.2024")
+		(rev "0.4.1")
 	)
 	(junction
